File: Hardware/Ultra-AV/ultra-AV.kicad_sch (KiCad schematic)
At the start: 16 parts, among them J1 Conn_01x04, J11 TC_1578891_SCART, J2 Conn_01x04, J3 Conn_01x04, J4 Conn_01x04, J5 Conn_01x04, J9 NorComp_111-014-213L001

Commit message: Redesigned VDP-board to include a socket, increased it to 4 layers. Various clean-ups here and there. Improved the printer-port and joystick-port 3D-models. Improved the cooling-fin 3D-model, and added attachment-spring in 3D-model.
Parts:
- J6: value (none) -> Conn_RCJ-023; footprint (none) -> LRJ:CUI_RCJ-023
- J7: value (none) -> Conn_RCJ-022
Changed lines of the file:
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@@
       (effects (font (size 1.27 1.27)) (justify left))
     )
-    (property "Value" "" (id 1) (at 177.8 31.0906 0)
+    (property "Value" "Conn_RCJ-023" (id 1) (at 177.8 31.0906 0)
       (effects (font (size 1.27 1.27)) (justify left) hide)
     )
-    (property "Footprint" "" (id 2) (at 171.45 41.91 0)
+    (property "Footprint" "LRJ:CUI_RCJ-023" (id 2) (at 171.45 41.91 0)
       (effects (font (size 1.27 1.27)) hide)
     )
@@
       (effects (font (size 1.27 1.27)) (justify left))
     )
-    (property "Value" "" (id 1) (at 177.8 53.9994 0)
+    (property "Value" "Conn_RCJ-022" (id 1) (at 177.8 53.9994 0)
       (effects (font (size 1.27 1.27)) (justify left) hide)
     )
