File: reference-projects/msx-cartridge-master/rom128k/rom128k.kicad_pcb (KiCad board)
At the start: 2 copper layers, 81.3 x 65.3 mm, 9 parts, among them J1 Conn_02x25_Odd_Even, SW1 DIPS_03, U1 74LS283, U2 SST39SF010

Commit message: Started remodelling the MSX cart-shells, as they don't seem to fit the cartridge-pcb's. Bit of clean-up in the directories.
Connections:
- net ~RD renamed ~{RD}
- net ~SLTSL renamed ~{SLTSL}
- J1 pad 1: Net-(J1-Pad1) -> unconnected-(J1-Pad1)
- J1 pad 10: Net-(J1-Pad10) -> unconnected-(J1-Pad10)
- J1 pad 11: Net-(J1-Pad11) -> unconnected-(J1-Pad11)
- J1 pad 12: Net-(J1-Pad12) -> unconnected-(J1-Pad12)
- J1 pad 13: Net-(J1-Pad13) -> unconnected-(J1-Pad13)
- J1 pad 15: Net-(J1-Pad15) -> unconnected-(J1-Pad15)
- J1 pad 16: Net-(J1-Pad16) -> unconnected-(J1-Pad16)
- J1 pad 2: Net-(J1-Pad2) -> unconnected-(J1-Pad2)
- J1 pad 3: Net-(J1-Pad3) -> unconnected-(J1-Pad3)
- J1 pad 42: Net-(J1-Pad42) -> unconnected-(J1-Pad42)
- J1 pad 48: Net-(J1-Pad48) -> unconnected-(J1-Pad48)
- J1 pad 49: Net-(J1-Pad49) -> unconnected-(J1-Pad49)
- J1 pad 5: Net-(J1-Pad5) -> unconnected-(J1-Pad5)
- J1 pad 50: Net-(J1-Pad50) -> unconnected-(J1-Pad50)
- J1 pad 6: Net-(J1-Pad6) -> unconnected-(J1-Pad6)
- J1 pad 7: Net-(J1-Pad7) -> unconnected-(J1-Pad7)
- J1 pad 8: Net-(J1-Pad8) -> unconnected-(J1-Pad8)
- J1 pad 9: Net-(J1-Pad9) -> unconnected-(J1-Pad9)
- U1 pad 10: Net-(U1-Pad10) -> unconnected-(U1-Pad10)
- U1 pad 9: Net-(U1-Pad9) -> unconnected-(U1-Pad9)
- U2 pad 1: Net-(U2-Pad1) -> unconnected-(U2-Pad1)
- U2 pad 30: Net-(U2-Pad30) -> unconnected-(U2-Pad30)
Other:
- net class Default removed
- net class Power removed
