File: Hardware/Ultra-MSX_Peripherals.kicad_sch (KiCad schematic)
At the start: 16 parts, among them J4 Amphenol_75869-306LF, J5 Ultra-IO-shield, J6 SDF-130J

Commit message: Added cooler and CPU-mount footprints, as well as Indication LEDs.
Connections:
- net RX1+ renamed SWDIO/RX1+
- net RX1- renamed SWDCLK/RX1-
- net RX2+ renamed nRESET/RX2+
- net RX2- renamed SWO/RX2-
- net SBU1/AUX1+ renamed VCT/SBU1
- net SBU2/AUX1- renamed GND/SBU2
Other:
- moved on the sheet: C12, J4, J6, JP1, R1, R28, R29, R34, R35, R39, R40, R41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

Commit message: Started fixing many small issues.
Parts:
- added CPU_Fan1, Sys_Fan1, Sys_Fan2: Molex_470533000, Connector:FanPinHeader_1x04_P2.54mm_Vertical, symbol LRJ-parts:Molex_470533000
Connections:
- net GNDA is gone; now on net GND: J5.54 (GND), J5.55 (GND)
- net +12V: now also CPU_Fan1.2, Sys_Fan1.2, Sys_Fan2.2
- net GND: now also CPU_Fan1.1, Sys_Fan1.1, Sys_Fan2.1
- net GND/SBU2: no longer names the net of J5.25 (AUX2-)
- net VCT/SBU1: no longer names the net of J5.24 (AUX1+)
- new net BLANK: J5.56 (BLANK)
- new net FanCtrl1: CPU_Fan1.4
- new net FanCtrl2: Sys_Fan1.4
- new net FanCtrl3: Sys_Fan2.4
- new net FanSen1: CPU_Fan1.3
- new net FanSen2: Sys_Fan1.3
- new net FanSen3: Sys_Fan2.3
- no-connect marks 2 -> 4
Other:
- note added: "Cooling Fans"
- note added: "Fan-headers"
- note added: "Header pinout: ----------- 1. GND 2. +12V 3. Tachometer/Sense 4. Control/PWM"
- note added: "https://blog.alexanderkoch.net/2020/01/making-of-fanboy.html http://pcbheaven.com/wikipages/How_PC_Fans_Work/"

Commit message: Updated the readme, silenced multiple errors in Kicad regarding simulation-files.
Parts:
- J6: Current rating (none) -> 1A; MPN (none) -> SDF-130J; Manufacturer (none) -> CUI Devices; Operating temperature (none) -> -40°C ~ 85°C; Status (none) -> OBSOLETE; Voltage rating (none) -> 100V
Changed lines of the file:
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@@
+      (effects (font (size 1.27 1.27)) hide)
+    )
+    (property "Sim.Enable" "0" (at 339.09 170.18 0)
       (effects (font (size 1.27 1.27)) hide)
     )
@@
       (effects (font (size 1.524 1.524)) (justify left) hide)
     )
+    (property "Sim.Enable" "0" (at 83.82 231.14 0)
+      (effects (font (size 1.27 1.27)) hide)
+    )
     (pin "1")
     (pin "2")
@@
       (effects (font (size 1.27 1.27)))
     )
+    (property "Sim.Enable" "0" (at 339.09 124.46 0)
+      (effects (font (size 1.27 1.27)) hide)
+    )
     (pin "1")
     (pin "2")
@@
     )
   )
-  (symbol (lib_name "Molex_470533000_2") (lib_id "LRJ-parts:Molex_470533000") (at 125.73 231.14 0) (unit 1)
+  (symbol (lib_id "LRJ-parts:Molex_470533000") (at 125.73 231.14 0) (unit 1)
     (in_bom yes) (on_board yes) (dnp no)
     (property "Reference" "Sys_Fan2" (at 123.19 220.98 0)
@@
       (effects (font (size 1.524 1.524)) (justify left) hide)
     )
+    (property "Sim.Enable" "0" (at 125.73 231.14 0)
+      (effects (font (size 1.27 1.27)) hide)
+    )
     (pin "1")
     (pin "2")
@@
     )
     (property "Datasheet" "https://www.cuidevices.com/product/resource/sdf-j.pdf" (at 342.011 43.18 0)
+      (effects (font (size 1.27 1.27)) hide)
+    )
+    (property "Sim.Enable" "0" (at 342.9 44.45 0)
+      (effects (font (size 1.27 1.27)) hide)
+    )
+    (property "Manufacturer" "CUI Devices" (at 317.5 31.75 0)
+      (effects (font (size 1.27 1.27)) hide)
+    )
+    (property "MPN" "SDF-130J" (at 317.5 34.29 0)
+      (effects (font (size 1.27 1.27)) hide)
+    )
+    (property "Description" "13 Position Circular Connector Receptacle, Female Socket, right angle" (at 287.02 49.53 0)
+      (effects (font (size 1.27 1.27)) hide)
+    )
+    (property "Status" "OBSOLETE" (at 317.5 52.07 0)
+      (effects (font (size 1.27 1.27)) hide)
+    )
+    (property "Voltage rating" "100V" (at 320.04 41.91 0)
+      (effects (font (size 1.27 1.27)) hide)
+    )
+    (property "Current rating" "1A" (at 320.04 36.83 0)
+      (effects (font (size 1.27 1.27)) hide)
+    )
+    (property "Operating temperature" "-40°C ~ 85°C" (at 314.96 39.37 0)
       (effects (font (size 1.27 1.27)) hide)
     )
@@
     )
   )
-  (symbol (lib_name "Molex_470533000_1") (lib_id "LRJ-parts:Molex_470533000") (at 105.41 231.14 0) (unit 1)
+  (symbol (lib_id "LRJ-parts:Molex_470533000") (at 105.41 231.14 0) (unit 1)
     (in_bom yes) (on_board yes) (dnp no)
     (property "Reference" "Sys_Fan1" (at 102.87 220.98 0)
@@
     (property "Status" "Active" (at 118.745 201.93 0)
       (effects (font (size 1.524 1.524)) (justify left) hide)
+    )
+    (property "Sim.Enable" "0" (at 105.41 231.14 0)
+      (effects (font (size 1.27 1.27)) hide)
     )
     (pin "1")
@@
       (effects (font (size 1.27 1.27)) hide)
     )
+    (property "Sim.Enable" "0" (at 34.29 95.25 0)
+      (effects (font (size 1.27 1.27)) hide)
+    )
