File: Hardware/Ultra-MSX_RAM.kicad_sch (KiCad schematic)
At the start: 11 parts, among them J10 Micro_SD_Card_Det_GCT, J13 TE_Conn_5822019-4, U10 SST39SF040, U8 AS6C8008-55ZIN

Commit message: Started fixing many small issues.
Parts:
- removed J13: TE_Conn_5822019-4, LRJ:SIMM-72_socket, symbol LRJ-parts:TE_Conn_5822019-4
- removed R36: R_ERJ-3GEYJ105V, Resistor_SMD:R_0603_1608Metric, symbol LRJ-parts:R_ERJ-3GEYJ105V
- added J9: Conn_SO-DIMM-144, LRJ:SODIMM-144_socket, symbol Ultra-MSX:Conn_SO-DIMM-144
Connections:
- net +3.3V: now also R38.1; no longer R38.2
- net +5V: now also J9.101 (VDD), J9.102 (VDD), J9.11 (VDD), J9.113 (VDD), J9.114 (VDD), J9.12 (VDD), J9.129 (VDD), J9.130 (VDD), J9.143 (VDD), J9.144 (VDD), J9.27 (VDD), J9.28 (VDD), J9.45 (VDD), J9.46 (VDD), J9.63 (VDD), J9.64 (VDD), J9.81 (VDD), J9.82 (VDD)
- net A17: now also J9.106 (BA0)
- net A18: now also J9.110 (BA1)
- net A19: now also J9.29 (A0)
- net A20: now also J9.30 (A3)
- net A21: now also J9.31 (A1)
- net A22: now also J9.32 (A4)
- net A23: now also J9.33 (A2)
- net A24: now also J9.34 (A5)
- net A25: now also J9.103 (A6)
- net A26: now also J9.104 (A7)
- net A27: now also J9.105 (A8)
- net A28: now also J9.109 (A9)
- net A29: now also J9.111 (A10)
- net A30: now also J9.112 (A11)
- net GND: now also J9.1 (VSS), J9.107 (VSS), J9.108 (VSS), J9.119 (VSS), J9.120 (VSS), J9.139 (VSS), J9.140 (VSS), J9.2 (VSS), J9.21 (VSS), J9.22 (VSS), J9.35 (VSS), J9.36 (VSS), J9.55 (VSS), J9.56 (VSS), J9.75 (VSS), J9.76 (VSS), J9.91 (VSS), J9.92 (VSS)
- net I2C_SCL: now also J9.141 (SDA)
- net I2C_SDA: now also J9.142 (SCL)
- net MCKE0: now also J9.62 (CKE0)
- net MCKE1: now also J9.68 (CKE1)
- net MD0: now also J9.3 (DQ0)
- net MD1: now also J9.5 (DQ1)
- net MD10: now also J9.41 (DQ10)
- net MD11: now also J9.43 (DQ11)
- net MD12: now also J9.47 (DQ12)
- net MD13: now also J9.49 (DQ13)
- net MD14: now also J9.51 (DQ14)
- net MD15: now also J9.53 (DQ15)
- net MD16: now also J9.83 (DQ16)
- net MD17: now also J9.85 (DQ17)
- net MD18: now also J9.87 (DQ18)
- net MD19: now also J9.89 (DQ19)
- net MD2: now also J9.7 (DQ2)
- net MD20: now also J9.93 (DQ20)
- net MD21: now also J9.95 (DQ21)
- net MD22: now also J9.97 (DQ22)
- net MD23: now also J9.99 (DQ23)
- net MD24: now also J9.121 (DQ24)
- net MD25: now also J9.123 (DQ25)
- net MD26: now also J9.125 (DQ26)
- net MD27: now also J9.127 (DQ27)
- net MD28: now also J9.131 (DQ28)
- net MD29: now also J9.133 (DQ29)
- net MD3: now also J9.9 (DQ3)
- net MD30: now also J9.135 (DQ30)
- net MD31: now also J9.137 (DQ31)
- net MD4: now also J9.13 (DQ4)
- net MD5: now also J9.15 (DQ5)
- net MD6: now also J9.17 (DQ6)
- net MD7: now also J9.19 (DQ7)
- net MD8: now also J9.37 (DQ8)
- net MD9: now also J9.39 (DQ9)
- net SD_DET_A: now also R37.1; no longer R38.1
- net SD_DET_B: now also R38.2; no longer R37.1
- net ~{CAS0}: now also J9.66 (~{CAS})
- net ~{MEM_WR}: now also J9.67 (~{WE})
- net ~{RAM_CS0}: now also U8.40 (CE2)
- net ~{RAM_CS1}: now also J9.71 (~{CS1})
- net ~{RAS0}: now also J9.65 (~{RAS})
- net ~{UMCS}: now also J9.69 (~{CS0})
- new net A31: J9.70 (A12)
- new net DQMB0: J9.23 (DQMB0)
- new net DQMB1: J9.25 (DQMB1)
- new net DQMB2: J9.115 (DQMB2)
- new net DQMB3: J9.117 (DQMB3)
- new net DQMB4: J9.24 (DQMB4)
- new net DQMB5: J9.26 (DQMB5)
- new net DQMB6: J9.116 (DQMB6)
- new net DQMB7: J9.118 (DQMB7)
- new net MCLK0: J9.61 (CK0)
- new net MCLK1: J9.74 (CK1)
- new net MD32: J9.4 (DQ32)
- new net MD33: J9.6 (DQ33)
- new net MD34: J9.8 (DQ34)
- new net MD35: J9.10 (DQ35)
- new net MD36: J9.14 (DQ36)
- new net MD37: J9.16 (DQ37)
- new net MD38: J9.18 (DQ38)
- new net MD39: J9.20 (DQ39)
- new net MD40: J9.38 (DQ40)
- new net MD41: J9.40 (DQ41)
- new net MD42: J9.42 (DQ42)
- new net MD43: J9.44 (DQ43)
- new net MD44: J9.48 (DQ44)
- new net MD45: J9.50 (DQ45)
- new net MD46: J9.52 (DQ46)
- new net MD47: J9.54 (DQ47)
- new net MD48: J9.84 (DQ48)
- new net MD49: J9.86 (DQ49)
- new net MD50: J9.88 (DQ50)
- new net MD51: J9.90 (DQ51)
- new net MD52: J9.94 (DQ52)
- new net MD53: J9.96 (DQ53)
- new net MD54: J9.98 (DQ54)
- new net MD55: J9.100 (DQ55)
- new net MD56: J9.122 (DQ56)
- new net MD57: J9.124 (DQ57)
- new net MD58: J9.126 (DQ58)
- new net MD59: J9.128 (DQ59)
- new net MD60: J9.132 (DQ60)
- new net MD61: J9.134 (DQ61)
- new net MD62: J9.136 (DQ62)
- new net MD63: J9.138 (DQ63)
- no-connect marks 0 -> 10
Other:
- note added: "3.3V SDRAM module, 100-133 MHz DDR2? EDO 5V, 32MB"
- note added: "MEMORY MAPPING: ---------------- - have 512K available for direct addressing in combination with the standard FC/FD/FE/FF ports - make another port available(which can accept 8bit,16bit, 32bit or even larger page numbers..fed sequentially) for some sub-switching to a larger memory. - to unload the processor with moving/clearing/copying one can add something as simple as a microcontroller to move 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"
- note added: "Memory-suggestions: ----------------------- Modern ---- IS42S16100H IS45S16100H Legacy ----"
- note removed: "Less common ram-sizes for SIMM-72 EDO ram include 128MB."
- moved on the sheet: C10, J10, JP3, R37, R38, R55, R80, U10A, U8A

Commit message: Updated the readme, silenced multiple errors in Kicad regarding simulation-files.
Parts:
- J9: symbol Ultra-MSX:Conn_SO-DIMM-144 -> LRJ-parts:Conn_SO-DIMM-144
Changed lines of the file:
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@@
+      (effects (font (size 1.27 1.27)) hide)
+    )
+    (property "Sim.Enable" "0" (at 57.15 64.77 0)
       (effects (font (size 1.27 1.27)) hide)
     )
@@
       (effects (font (size 1.27 1.27)) hide)
     )
+    (property "Sim.Enable" "0" (at 334.01 43.18 0)
+      (effects (font (size 1.27 1.27)) hide)
+    )
     (pin "1")
     (pin "10")
@@
     )
   )
-  (symbol (lib_id "Ultra-MSX:Conn_SO-DIMM-144") (at 166.37 118.11 0) (unit 1)
+  (symbol (lib_id "LRJ-parts:Conn_SO-DIMM-144") (at 166.37 118.11 0) (unit 1)
     (in_bom yes) (on_board yes) (dnp no)
     (property "Reference" "J9" (at 167.64 38.1 0)
@@
     )
     (property "Frequency" "133MHz" (at 204.47 113.03 0)
+      (effects (font (size 1.27 1.27)) hide)
+    )
+    (property "Sim.Enable" "0" (at 166.37 118.11 0)
       (effects (font (size 1.27 1.27)) hide)
     )
@@
       (effects (font (size 1.27 1.27)) hide)
     )
+    (property "Sim.Enable" "0" (at 57.15 154.94 0)
+      (effects (font (size 1.27 1.27)) hide)
+    )
     (pin "15")
     (pin "16")
@@
       (effects (font (size 1.27 1.27)) hide)
     )
+    (property "Sim.Enable" "0" (at 26.67 74.93 0)
+      (effects (font (size 1.27 1.27)) hide)
+    )
