File: Hardware/Ultra-VDP/Ultra-VDP.kicad_sch (KiCad schematic)
At the start: 95 parts, among them J1 BC075-05, J2 BC075-10, J3 CBUS, J4 BC075-10, J5 BC075-06, J6 BC075-10, J7 BC075-10, J8 BC075-05, U14 V53C8125HT30, U3 V9958, U6 LMH1980, Y1 21.477270MHz, Y3 4.433618MHz

Commit message: Many tweaks and changes, such as a slight redesign of the VDP-baord.
Parts:
- removed trace1, trace10, trace11, trace12, trace13, trace14, trace15, trace16, trace17, trace18, trace19, trace2, trace20, trace21, trace3, trace4, trace5, trace6, trace7, trace8, trace9: pcb-trace, LRJ:NetTie-2_SMD_Pad0.2mm, symbol LRJ-parts:Trace
- added trace1, trace10, trace11, trace12, trace13, trace14, trace15, trace16, trace17, trace18, trace19, trace2, trace20, trace21, trace22, trace3, trace4, trace6, trace7, trace8, trace9: pcb-trace, LRJ:NetTie-2_SMD_Pad0.2mm, symbol LRJ-parts:Trace_0.2mm
- C12, C19: value 47pF -> C_CC0603JRNPO9BN470; symbol Device:C -> LRJ-parts:C_CC0603JRNPO9BN470; Capacitance (none) -> 47pF; MPN (none) -> CC0603JRNPO9BN470; Manufacturer (none) -> Yageo; Mounting type (none) -> SMD; Operating Temperature (none) -> -55°C ~ 125°C; Status (none) -> Active; Temperature Coefficient  (none) -> C0G; Voltage rating (none) -> 50V
- JP5: now left out of the parts list
- R10, R13, R14, R15: value 75 -> R_ERJ-PA3F75R0V; footprint Resistor_SMD:R_0603_1608Metric -> LRJ:R_0603_1608Metric_roundcourt; symbol Device:R -> LRJ-parts:R_ERJ-PA3F75R0V; Current rating (none) -> n/a; MPN (none) -> ERJ-PA3F75R0V; Manufacturer (none) -> Panasonic Electronic Components; Mounting type (none) -> SMD; Operating Temperature  (none) -> -55°C to +155°C; Resistance (none) -> 75Ω; Status (none) -> Active; Temperature coeffecient (none) -> ±100ppm/°C; Voltage rating (none) -> 49V
- R12, R27, R5, R6, R61, R8: value 100 -> R_CRGP0603F220R; symbol Device:R -> LRJ-parts:R_CRG0603F100R; MPN (none) -> CRGP0603F220R; Manufacturer (none) -> TE Connectivity; Operating Temperature  (none) -> -55°C to 125°C; Power (Watts)  (none) -> 0.1W, 1/10W; Resistance (none) -> 100Ω; Status (none) -> Active
- R3: value 1k -> R_ERA-3VRW1001V; footprint Resistor_SMD:R_0603_1608Metric -> Resistor_SMD:R_0603_1608Metric_Pad0.98x0.95mm_HandSolder; symbol Device:R -> LRJ-parts:R_ERA-3VRW1001V; Details (none) -> https://na.industrial.panasonic.com/products/resistors/smd-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; MPN (none) -> ERA-3VRW1001V; Manufacturer (none) -> Panasonic; Operating temperature (none) -> -55C to +155C; Resistance (none) -> 1kΩ; Status (none) -> Active; Tolerance (none) -> ±0.05%; Voltage rating (none) -> 75V
- R4: value 1M -> R_ERJ-3GEYJ105V; footprint Resistor_SMD:R_0805_2012Metric -> Resistor_SMD:R_0603_1608Metric; symbol Device:R -> LRJ-parts:R_ERJ-3GEYJ105V; MPN (none) -> ERJ-3GEYJ105V; Manufacturer (none) -> Panasonic Electronic Components; Mounting type (none) -> SMD; Operating Temperature  (none) -> -55°C to +155°C; Resistance (none) -> 1MΩ; Status (none) -> Active; Voltage rating (none) -> 75V
- Y1: value 21.477270MHz -> Y_HCM4921477270ABJT; footprint Ultra-MSX:Crystal_HC-49U_Vert -> LRJ:Crystal_HC49-US_Vertical; symbol Device:Crystal -> LRJ-parts:Y_HCM4921477270ABJT; Frequency (none) -> 21.47727MHz; Manufacturer (none) -> Citizen Finedevice Co Ltd; Status (none) -> Active
- Y3: value 4.433618MHz -> Y_ECS-44-20-4X; footprint Ultra-MSX:Crystal_HC-49U_Vert -> LRJ:Crystal_HC49-US_Vertical_THT; symbol Device:Crystal -> LRJ-parts:Y_ECS-44-20-4X; Frequency (none) -> 4.433618MHz; MPN (none) -> ECS-44-20-4X; Manufacturer (none) -> ECS; Operating temperature (none) -> -10 C ~ +70 C; Resistance (none) -> 150R; Status (none) -> Active
Connections:
- net A2: now also trace9.1
- net A3: now also trace10.1
- net A4: now also trace11.1
- net A5: now also trace12.1
- net A6: now also trace13.1
- net A7: now also trace14.1
- net A8: now also trace15.1
- net BLANK: now also J5.6 (Pin_6), trace4.1
- net BLUE2: now also R15.1; no longer R15.2
- net COMPSYNC: now also R10.2; no longer R10.1
- net D10: now also trace2.1
- net D11: now also trace3.1
- net D12: now also trace18.1
- net D13: now also trace6.1
- net D14: now also trace7.1
- net D15: now also trace8.1
- net D8: now also trace17.1
- net D9: now also trace16.1
- net GND: now also R10.1; no longer R10.2
- net GREEN2: now also R14.1; no longer R14.2
- net PAL_CLK_IN+: now also R4.1; no longer R4.2
- net PAL_CLK_IN-: now also R3.2; no longer R3.1
- net RED2: now also R13.1; no longer R13.2
- net TCK: now also trace21.1
- net TDI: now also trace20.1
- net TDO: now also trace22.1
- net TMS: now also trace19.1
- net VREF: now also trace1.1
- net B-Main renamed B-Mb
- net B-Mb: now also R15.2; no longer R15.1
- net G-Main renamed G-Mb
- net G-Mb: now also R14.2; no longer R14.1
- net R-Main renamed R-Mb
- net R-Mb: now also R13.2; no longer R13.1
- new net: R3.1, R4.2
Other:
- note added: "Connects to large caps on motherboard."
- note added: "Note: these pins are only in use (on the Motherboard) when utilizing a more advanced VDP such as V9990, or F18A. ->"
- note removed: "Connects to large caps on mainboard."
- note removed: "Note: these pins are only in use when utilizing a more advanced VDP such as V9990, or F18A. ->"
- moved on the sheet: R1, R10, R12, R13, R14, R15, R27, R3, R4, R55, R56, R57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
